File: x60/_autosave-x60.sch (KiCad schematic (older format))
At the start: 141 parts, among them SW1 SW_Push, U1 ATmega32U4-AU, Y1 16mhz

Commit message: arranged the keys on the pcb
Parts:
- MX61: footprint MX_Only:MXOnly-1U-NoLED -> MX_Only:MXOnly-1.5U-NoLED
Changed lines of the file:
@@
 F 0 "MX61" H 11633 1573 60  0000 C CNN
 F 1 "\\" H 11633 1499 20  0000 C CNN
-F 2 "MX_Only:MXOnly-1U-NoLED" H 10975 1325 60  0001 C CNN
+F 2 "MX_Only:MXOnly-1.5U-NoLED" H 10975 1325 60  0001 C CNN
 F 3 "" H 10975 1325 60  0001 C CNN
 	1    11600 1350
