File: x60Rev.1/x60.kicad_pcb (KiCad board)
At the start: 2 copper layers, 281 x 92.9 mm, 154 parts, among them J1 USB_C_Receptacle_USB2.0, SW1 SW_Push, U1 ATmega32U4-AU, Y1 16mhz

Commit message: generated production files
Routing:
- net COL11: track 235.1 -> 238.8 mm
Other:
- rule pad_to_mask_clearance: 0.051 -> 0

Commit message: updated components
Parts:
- SW1: footprint random-keyboard-parts:SKQG-1155865 -> random-keyboard-parts:SKQGADE010
