File: x60Rev.1/x60.sch (KiCad schematic (older format))
At the start: 154 parts, among them J1 USB_C_Receptacle_USB2.0, SW1 SW_Push, U1 ATmega32U4-AU, Y1 16mhz

Commit message: updated components
Parts:
- SW1: footprint random-keyboard-parts:SKQG-1155865 -> random-keyboard-parts:SKQGADE010
Changed lines of the file:
@@
 F 0 "SW1" H 4575 5560 50  0000 C CNN
 F 1 "SW_Push" H 4575 5469 50  0000 C CNN
-F 2 "random-keyboard-parts:SKQG-1155865" H 4575 5475 50  0001 C CNN
+F 2 "random-keyboard-parts:SKQGADE010" H 4575 5475 50  0001 C CNN
 F 3 "~" H 4575 5475 50  0001 C CNN
 	1    4575 5275
